File: PCB/main/main.kicad_sch (KiCad schematic)
At the start: 56 parts, among them J1 Conn_01x05, J2 USB_C_Receptacle_USB2.0_16P, J3 Conn_01x03_Pin, J6 Conn_01x05, SW1 Reset, SW2 Boot, U2 AMS1117-3.3, U4 RP2040, U5 L9110, U6 MX25L3233FM, Y1 ABM8G-12.000MHZ-D2Y-T

Commit message: Started new branch
Parts:
- removed C3, C5: 1u, symbol Device:C
- removed C4, C6, C9: 100n, symbol Device:C
- removed J3: Conn_01x03_Pin, symbol Connector:Conn_01x03_Pin
- removed R1, R2: 27.4, symbol Device:R
- removed R7: 1k, symbol Device:R
- removed R8: 10k, symbol Device:R
- removed TP1: 10, symbol Connector:TestPoint
- removed TP10: 19, symbol Connector:TestPoint
- removed TP11: 20, symbol Connector:TestPoint
- removed TP12: 21, symbol Connector:TestPoint
- removed TP13: 22, symbol Connector:TestPoint
- removed TP14: 23, symbol Connector:TestPoint
- removed TP15: 25, symbol Connector:TestPoint
- removed TP16: 6, symbol Connector:TestPoint
- removed TP17: 7, symbol Connector:TestPoint
- removed TP2: 11, symbol Connector:TestPoint
- removed TP3: 12, symbol Connector:TestPoint
- removed TP4: 13, symbol Connector:TestPoint
- removed TP5: 14, symbol Connector:TestPoint
- removed TP6: 15, symbol Connector:TestPoint
- removed TP7: 16, symbol Connector:TestPoint
- removed TP8: 17, symbol Connector:TestPoint
- removed TP9: 18, symbol Connector:TestPoint
- removed U4: RP2040, Package_DFN_QFN:QFN-56-1EP_7x7mm_P0.4mm_EP3.2x3.2mm, symbol MCU_RaspberryPi:RP2040
- removed U6: MX25L3233FM, Package_SO:SOIC-16W_7.5x10.3mm_P1.27mm, symbol Memory_Flash:MX25L3233FM
- added U1: (no value), EasyEDA_Lib:TSSOP-20_L6.5-W4.4-P0.65-LS6.4-BL, symbol EasyEDA_Lib:PY32F003F18P6TU
Connections:
- net +5V: now also U1.9 (VCC)
- net GND: now also U1.7 (VSS)
- net GPIO0 renamed TX_UP
- net GPIO1 renamed RX_UP
- net GPIO4 renamed Touch
- net GPIO8 renamed TX_DOWN
- net GPIO9 renamed RX_DOWN
- new net OSCIN: U1.16 (PF0-OSCIN)
- new net OSCOUT: U1.17 (PF1-OSCOUT)
Other:
- note removed: "Extra GPIO"
- note removed: "QSPI Flash"

Commit message: Progress on schematic
Parts:
- removed C1: 100n, symbol Device:C
- removed C10, C11: 15p, symbol Device:C
- removed C12, C13: 10u, symbol Device:C
- removed C7: C, Capacitor_SMD:C_1206_3216Metric_Pad1.33x1.80mm_HandSolder, symbol Device:C
- removed C8: 4.7nF, symbol Device:C_Small
- removed D1, D2: D_Schottky, symbol Device:D_Schottky
- removed J2: USB_C_Receptacle_USB2.0_16P, Connector_USB:USB_C_Receptacle_GCT_USB4110, symbol Connector:USB_C_Receptacle_USB2.0_16P
- removed R10: 10k, symbol Device:R
- removed R11: 15k, symbol Device:R
- removed R4: 1M, symbol Device:R
- removed R5, R6: 5.1k, symbol Device:R
- removed R9: 1k, symbol Device:R
- removed SW1: Reset, symbol Switch:SW_Push
- removed SW2: Boot, symbol Switch:SW_Push
- removed U2: AMS1117-3.3, Package_TO_SOT_SMD:SOT-223-3_TabPin2, symbol Regulator_Linear:AMS1117-3.3
- removed Y1: ABM8G-12.000MHZ-D2Y-T, CRYSTAL_ABM8G_ABR, symbol 2026-04-12_02-59-10:ABM8G-12.000MHZ-D2Y-T
- added C2, C5, C7, C8: 100nF, PCM_JLCPCB:C_0402, symbol PCM_JLCPCB-Capacitors:0402,100nF
- added C3, C4: 10uF, PCM_JLCPCB:C_0805, symbol PCM_JLCPCB-Capacitors:0805,10uF
- added R1: 10kΩ, PCM_JLCPCB:R_0402, symbol PCM_JLCPCB-Resistors:0402,10kΩ
- added S1, S2: Tactile Button, 160gf, PCM_JLCPCB:SW_TS-1088-AR02016, symbol PCM_JLCPCB-Connectors_Buttons:Tactile Button, 160gf, 12V, 50mA, 4.0mm
Connections:
- net +3.3V is gone; now on net +5V: U3.2 (Pot+), U7.5 (VDD)
- net GPIO2 is gone; now on net M1: U5.6 (IA)
- net GPIO26_ADC0 is gone; now on net Wiper: U3.3 (PotW)
- net GPIO3 is gone; now on net M2: U5.7 (IB)
- net GPIO5 is gone; now on net RGB_DIN: R12.1
- net OSCOUT is gone; now on net Touch: U1.17 (PF1-OSCOUT)
- net +5V: now also C4.1, C5.1, C7.1, C8.1, R1.1, S2.1 (A)
- net BOOT_BTN: now also U1.15 (PF4-BOOT0), S2.2 (B)
- net GND: now also C2.2, C3.2, C4.2, C5.2, C7.2, C8.2, R1.2, S1.1 (A)
- net RX_DOWN: now also U1.20 (PA1)
- net RX_UP: now also U1.2 (PA3)
- net TX_DOWN: now also U1.19 (PA0)
- net TX_UP: now also U1.1 (PA2)
- net VMOT: now also C3.1
- net SWD: now reaches U1.10 (PA13-SWD)
- net SWC: now reaches U1.11 (PA14-SWC)
- net RUN_BTN: now reaches U1.18 (PF2-NRST)
- net RUN_BTN: now also C2.1, S1.2 (B)
- net Wiper: now reaches U1.3 (PA4)
- net RGB_DIN: now reaches U1.4 (PA5)
- net M1: now reaches U1.5 (PA6)
- net M2: now reaches U1.6 (PA7)
- net OSCIN: no longer names the net of U1.16 (PF0-OSCIN)
- no-connect marks 2 -> 0
Other:
- note removed: "USB"
- note removed: "Voltage regulator (optional through hole for master device) or maybe solder jumper"
- moved on the sheet: U1

Commit message: PCB Nearly Complete
Parts:
- removed R12: 470, symbol Device:R
- added J2: Conn_01x05_Pin, symbol Connector:Conn_01x05_Pin
- added R2: 470Ω, PCM_JLCPCB:R_0402, symbol PCM_JLCPCB-Resistors:0402,470Ω
- U3: footprint Motorized Fader:MF60T -> Faders:MF60T-MF100T
- U5: footprint (none) -> L9110:so-8
Connections:
- net +5V: now also J2.1 (Pin_1); no longer R1.1
- net BOOT_BTN: now also R1.1
- net GND: now also J2.4 (Pin_4)
- net RGB_DIN: now also R2.1
- net SWC: now also J2.3 (Pin_3)
- net SWD: now also J2.2 (Pin_2)
- net at D3.4 (DI): now also R2.2
- net RUN_BTN renamed NRST
- net NRST: now also J2.5 (Pin_5)

Commit message: PCB Updates
Parts:
- added J3: Boot Pin, symbol Connector:Conn_01x01_Pin
Connections:
- net BOOT_BTN: now also J3.1 (Pin_1)
- net GND: now also J1.5 (Pin_5), J6.5 (Pin_5); no longer J1.1 (Pin_1), J6.1 (Pin_1)
- net RX_DOWN: now also J6.1 (Pin_1); no longer J6.5 (Pin_5)
- net RX_UP: now also J1.2 (Pin_2); no longer J1.4 (Pin_4)
- net TX_DOWN: now also J6.2 (Pin_2); no longer J6.4 (Pin_4)
- net TX_UP: now also J1.1 (Pin_1); no longer J1.5 (Pin_5)
- net VMOT: now also J1.4 (Pin_4), J6.4 (Pin_4); no longer J1.2 (Pin_2), J6.2 (Pin_2)
Other:
- moved on the sheet: J1, J6
Changed lines of the file:
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@@
 		)
 	)
+	(global_label "BOOT_BTN"
+		(shape input)
+		(at 181.61 107.95 0)
+		(fields_autoplaced yes)
+		(effects
+			(font
+				(size 1.27 1.27)
+			)
+			(justify left)
+		)
+		(property "Intersheetrefs" "${INTERSHEET_REFS}"
+			(at 194.0295 107.95 0)
+			(hide yes)
+			(show_name no)
+			(do_not_autoplace no)
+			(effects
+				(font
+					(size 1.27 1.27)
+				)
+				(justify left)
+			)
+		)
+	)
 	(global_label "RGB_DIN"
 		(shape input)
@@
 	)
 	(symbol
+		(lib_id "Connector:Conn_01x01_Pin")
+		(at 176.53 107.95 0)
+		(unit 1)
+		(body_style 1)
+		(exclude_from_sim no)
+		(in_bom yes)
+		(on_board yes)
+		(in_pos_files yes)
+		(dnp no)
+		(fields_autoplaced yes)
+		(property "Reference" "J3"
+			(at 177.165 102.87 0)
+			(show_name no)
+			(do_not_autoplace no)
+			(effects
+				(font
+					(size 1.27 1.27)
+				)
+			)
+		)
+		(property "Value" "Boot Pin"
+			(at 177.165 105.41 0)
+			(show_name no)
+			(do_not_autoplace no)
+			(effects
+				(font
+					(size 1.27 1.27)
+				)
+			)
+		)
+		(property "Footprint" ""
+			(at 176.53 107.95 0)
+			(hide yes)
+			(show_name no)
+			(do_not_autoplace no)
+			(effects
+				(font
+					(size 1.27 1.27)
+				)
+			)
+		)
+		(property "Datasheet" ""
+			(at 176.53 107.95 0)
+			(hide yes)
+			(show_name no)
+			(do_not_autoplace no)
+			(effects
+				(font
+					(size 1.27 1.27)
+				)
+			)
+		)
+		(property "Description" "Generic connector, single row, 01x01, script generated"
+			(at 176.53 107.95 0)
+			(hide yes)
+			(show_name no)
+			(do_not_autoplace no)
+			(effects
+				(font
+					(size 1.27 1.27)
+				)
+			)
+		)
+		(pin "1"
+		)
+		(instances
+			(project "main"
+				(path "/90b10b66-12e8-465c-a51a-726ddba72d44"
+					(reference "J3")
+					(unit 1)
+				)
+			)
+		)
+	)
+	(symbol
 		(lib_id "Connector:Conn_01x05_Pin")
 		(at 144.78 130.81 0)
@@
 	(symbol
 		(lib_id "Connector_Generic:Conn_01x05")
-		(at 24.13 104.14 0)
-		(mirror y)
+		(at 24.13 104.14 180)
 		(unit 1)
 		(body_style 1)
@@
 		(in_pos_files yes)
 		(dnp no)
-		(fields_autoplaced yes)
 		(property "Reference" "J1"
-			(at 24.13 92.71 0)
+			(at 24.13 115.57 0)
 			(show_name no)
 			(do_not_autoplace no)
@@
 		)
 		(property "Value" "Conn_01x05"
-			(at 24.13 95.25 0)
+			(at 24.13 113.03 0)
 			(show_name no)
 			(do_not_autoplace no)
@@
 	(symbol
 		(lib_id "Connector_Generic:Conn_01x05")
-		(at 24.13 135.89 0)
-		(mirror y)
+		(at 24.13 135.89 180)
 		(unit 1)
 		(body_style 1)
@@
 		(in_pos_files yes)
 		(dnp no)
-		(fields_autoplaced yes)
 		(property "Reference" "J6"
-			(at 24.13 124.46 0)
+			(at 24.13 147.32 0)
 			(show_name no)
 			(do_not_autoplace no)
@@
 		)
 		(property "Value" "Conn_01x05"
-			(at 24.13 127 0)
+			(at 24.13 144.78 0)
 			(show_name no)
 			(do_not_autoplace no)
