File: PCB/main/main.kicad_sch (KiCad schematic)
At the start: 19 parts, among them J1 Conn_01x05, J2 Conn_01x05_Pin, J3 Boot Pin, J6 Conn_01x05, U5 L9110

Commit message: Set components to DNP
Parts:
- J1, J2, J6: now not fitted; now left out of the parts list
- J3: footprint (none) -> Connector_PinHeader_2.54mm:PinHeader_1x01_P2.54mm_Vertical; now not fitted; now left out of the parts list
Changed lines of the file:
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@@
 		(body_style 1)
 		(exclude_from_sim no)
-		(in_bom yes)
+		(in_bom no)
 		(on_board yes)
-		(in_pos_files yes)
-		(dnp no)
+		(in_pos_files no)
+		(dnp yes)
 		(fields_autoplaced yes)
 		(property "Reference" "J3"
@@
 			)
 		)
-		(property "Footprint" ""
+		(property "Footprint" "Connector_PinHeader_2.54mm:PinHeader_1x01_P2.54mm_Vertical"
 			(at 176.53 107.95 0)
 			(hide yes)
@@
 		(body_style 1)
 		(exclude_from_sim no)
-		(in_bom yes)
+		(in_bom no)
 		(on_board yes)
-		(in_pos_files yes)
-		(dnp no)
+		(in_pos_files no)
+		(dnp yes)
 		(fields_autoplaced yes)
 		(property "Reference" "J2"
@@
 		(body_style 1)
 		(exclude_from_sim no)
-		(in_bom yes)
+		(in_bom no)
 		(on_board yes)
-		(in_pos_files yes)
-		(dnp no)
+		(in_pos_files no)
+		(dnp yes)
 		(property "Reference" "J1"
 			(at 24.13 115.57 0)
@@
 		(body_style 1)
 		(exclude_from_sim no)
-		(in_bom yes)
+		(in_bom no)
 		(on_board yes)
-		(in_pos_files yes)
-		(dnp no)
+		(in_pos_files no)
+		(dnp yes)
 		(property "Reference" "J6"
 			(at 24.13 147.32 0)

Commit message: Progress on PCB
Flipped side of board for components
Parts:
- removed J2: Conn_01x05_Pin, symbol Connector:Conn_01x05_Pin
- removed J3: Boot Pin, Connector_PinHeader_2.54mm:PinHeader_1x01_P2.54mm_Vertical, symbol Connector:Conn_01x01_Pin
- added J4: Conn_01x06_Pin, Connector_PinHeader_2.54mm:PinHeader_1x06_P2.54mm_Vertical, symbol Connector:Conn_01x06_Pin
Connections:
- net +5V: now also J4.1 (Pin_1)
- net GND: now also J4.6 (Pin_6)
- net NRST: now also J4.4 (Pin_4)
- net SWC: now also J4.3 (Pin_3)
- net SWD: now also J4.2 (Pin_2)
- net BOOT_BTN renamed BOOT
- net BOOT: now also J4.5 (Pin_5)
