File: PCB/main/main.kicad_sch (KiCad schematic)
At the start: 18 parts, among them J1 Conn_01x05, J4 Conn_01x06_Pin, J6 Conn_01x05, U5 L9110

Commit message: Renamed code folder to firmware, added motor test + comments
Parts:
- U1: Actual part number (none) -> PY32F003F18P6TU; LCSC (none) -> C5379864; Manufacturer Part PY32F003F18P6TU -> (none); Part (none) -> PY32F003F18P6TU; Supplier Part C5379864 -> (none)
Changed lines of the file:
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@@
 			)
 		)
-		(property "Manufacturer Part" "PY32F003F18P6TU"
+		(property "Part" "PY32F003F18P6TU"
 			(at 144.78 95.25 0)
 			(hide yes)
@@
 			)
 		)
-		(property "Supplier Part" "C5379864"
+		(property "LCSC" "C5379864"
 			(at 144.78 95.25 0)
 			(hide yes)
@@
 			(at 144.78 95.25 0)
 			(hide yes)
+			(show_name no)
+			(do_not_autoplace no)
+			(effects
+				(font
+					(size 1.27 1.27)
+				)
+			)
+		)
+		(property "Actual part number" "PY32F003F18P6TU"
+			(at 144.78 95.25 0)
+			(hide yes)
