File: PCB/main/main.kicad_pcb (KiCad board)
At the start: 2 copper layers, 17 x 101.3 mm, 18 parts, among them J1 Conn_01x05, J4 Conn_01x06_Pin, J6 Conn_01x05, U5 L9110

Commit message: Renamed code folder to firmware, added motor test + comments
Changed lines of the file:
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@@
 			(at 0 15.08 90)
 			(layer "F.Fab")
+			(hide yes)
 			(effects
 				(font
@@
 			(at 5 -4.6 270)
 			(layer "B.Fab")
+			(hide yes)
 			(effects
 				(font
@@
 		(layer "F.SilkS")
 		(effects
+			(font
+				(size 0.6 0.6)
+				(thickness 0.15)
+				(bold yes)
+			)
+			(justify left bottom)
+		)
+	)
+	(gr_text "https://github.com/PKCubed/OpenFader"
+		(at 150.1 162.5 90)
+		(layer "F.SilkS")
+		(effects
